File: hardware/riffle-0.2.sch (EAGLE design)
At the start: 32 parts, among them IC1 ATMEGA328P, IC2 MCP73831, IC3 CH340G, IC4 MCP1700-33, IC5 24AA128SN, J1 AYZ0202, X1 USBSMD, X2 12MHz, X3 16 MHz

Commit message: update
Parts:
- added C8: .1u, resistor:C-EUC0805
- added JP4: (no value), SparkFun-Connectors:M07
- added REMOTE: FDN340P, zetex:PMOSSOT23
Connections:
- new net N$7: C8.2, JP4.7, REMOTE.D
- net A0: now also JP4.2
- net A1: now also JP4.3
- net D2: now also JP4.4
- net D4: now also REMOTE.G
- net GND: now also C8.1, JP4.1
- net SCL: now also JP4.6
- net SDA: now also JP4.5
- net VCC: now also REMOTE.S
Changed lines of the file:
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@@
 <part name="RTCINT" library="_SparkFun" deviceset="SOLDERJUMPER" device="NO"/>
 <part name="X3" library="SparkFun" deviceset="RESONATOR" device="SMD" value="16 MHz"/>
+<part name="REMOTE" library="zetex" deviceset="PMOSSOT23" device="" value="FDN340P"/>
+<part name="GND1" library="SparkFun" deviceset="GND" device=""/>
+<part name="P+6" library="supply1" deviceset="VCC" device=""/>
+<part name="C8" library="resistor" deviceset="C-EU" device="C0805" value=".1u"/>
+<part name="JP4" library="SparkFun-Connectors" deviceset="M07" device=""/>
 </parts>
 <sheets>
@@
 </instance>
 <instance part="X3" gate="G$1" x="10.16" y="41.91" rot="R270"/>
+<instance part="REMOTE" gate="A" x="140.462" y="41.148" rot="MR270"/>
+<instance part="GND1" gate="1" x="118.618" y="41.148" rot="R270"/>
+<instance part="P+6" gate="VCC" x="150.876" y="43.688"/>
+<instance part="C8" gate="G$1" x="125.476" y="41.148" smashed="yes" rot="R90">
+<attribute name="NAME" x="125.095" y="42.672" size="1.778" layer="95" rot="R90"/>
+<attribute name="VALUE" x="128.397" y="47.244" size="1.778" layer="96" rot="R270"/>
+</instance>
+<instance part="JP4" gate="G$1" x="162.56" y="18.034" rot="R180"/>
 </instances>
 <busses>
@@
 <pinref part="BAT" gate="G$1" pin="-"/>
 </segment>
+<segment>
+<pinref part="GND1" gate="1" pin="GND"/>
+<wire x1="121.158" y1="41.148" x2="122.936" y2="41.148" width="0.1524" layer="91"/>
+<pinref part="C8" gate="G$1" pin="1"/>
+</segment>
+<segment>
+<wire x1="157.48" y1="23.114" x2="145.796" y2="23.114" width="0.1524" layer="91"/>
+<label x="143.764" y="23.876" size="1.778" layer="95"/>
+<pinref part="JP4" gate="G$1" pin="1"/>
+</segment>
 </net>
 <net name="VBUS" class="1">
@@
 <wire x1="62.23" y1="62.23" x2="76.2" y2="62.23" width="0.1524" layer="91"/>
 <label x="66.04" y="62.23" size="1.778" layer="95"/>
+</segment>
+<segment>
+<wire x1="157.48" y1="20.574" x2="145.796" y2="20.574" width="0.1524" layer="91"/>
+<label x="140.716" y="20.574" size="1.778" layer="95"/>
+<pinref part="JP4" gate="G$1" pin="2"/>
 </segment>
 </net>
@@
 <pinref part="RTC" gate="G$1" pin="VCC"/>
 </segment>
+<segment>
+<pinref part="REMOTE" gate="A" pin="S"/>
+<pinref part="P+6" gate="VCC" pin="VCC"/>
+<wire x1="150.876" y1="41.148" x2="145.542" y2="41.148" width="0.1524" layer="91"/>
+</segment>
 </net>
 <net name="AREF" class="0">
@@
 <label x="66.04" y="29.21" size="1.778" layer="95"/>
 </segment>
+<segment>
+<pinref part="REMOTE" gate="A" pin="G"/>
+<wire x1="143.002" y1="46.228" x2="142.748" y2="50.038" width="0.1524" layer="91"/>
+<label x="141.986" y="52.832" size="1.778" layer="95"/>
+</segment>
 </net>
 <net name="D8" class="0">
@@
 <wire x1="62.23" y1="59.69" x2="78.74" y2="59.69" width="0.1524" layer="91"/>
 <label x="66.04" y="59.69" size="1.778" layer="95"/>
+</segment>
+<segment>
+<wire x1="157.48" y1="18.034" x2="146.558" y2="18.034" width="0.1524" layer="91"/>
+<label x="141.478" y="18.034" size="1.778" layer="95"/>
+<pinref part="JP4" gate="G$1" pin="3"/>
 </segment>
 </net>
@@
 <label x="-72.39" y="21.59" size="1.778" layer="95"/>
 </segment>
+<segment>
+<wire x1="157.48" y1="15.494" x2="146.304" y2="15.494" width="0.1524" layer="91"/>
+<wire x1="146.304" y1="15.494" x2="146.304" y2="15.24" width="0.1524" layer="91"/>
+<label x="143.002" y="15.24" size="1.778" layer="95"/>
+<pinref part="JP4" gate="G$1" pin="4"/>
+</segment>
 </net>
 <net name="D10" class="0">
@@
 <label x="13.208" y="163.83" size="1.778" layer="95"/>
 </segment>
+<segment>
+<wire x1="157.48" y1="12.954" x2="144.018" y2="12.954" width="0.1524" layer="91"/>
+<wire x1="144.018" y1="12.954" x2="144.018" y2="13.462" width="0.1524" layer="91"/>
+<label x="140.208" y="12.954" size="1.778" layer="95"/>
+<pinref part="JP4" gate="G$1" pin="5"/>
+</segment>
 </net>
 <net name="SCL" class="0">
@@
 <pinref part="RTC" gate="G$1" pin="SCL"/>
 <label x="12.954" y="166.878" size="1.778" layer="95"/>
+</segment>
+<segment>
+<pinref part="JP4" gate="G$1" pin="6"/>
+<wire x1="157.48" y1="10.414" x2="150.622" y2="10.414" width="0.1524" layer="91"/>
+<label x="148.336" y="10.414" size="1.778" layer="95"/>
 </segment>
 </net>
@@
 </segment>
 </net>
+<net name="N$7" class="0">
+<segment>
+<pinref part="REMOTE" gate="A" pin="D"/>
+<wire x1="135.382" y1="41.148" x2="133.858" y2="41.148" width="0.1524" layer="91"/>
+<wire x1="133.858" y1="41.148" x2="133.858" y2="7.366" width="0.1524" layer="91"/>
+<pinref part="JP4" gate="G$1" pin="7"/>
+<wire x1="133.858" y1="7.366" x2="157.48" y2="7.366" width="0.1524" layer="91"/>
+<wire x1="157.48" y1="7.366" x2="157.48" y2="7.874" width="0.1524" layer="91"/>
+<pinref part="C8" gate="G$1" pin="2"/>
+<wire x1="133.858" y1="41.148" x2="130.556" y2="41.148" width="0.1524" layer="91"/>
+<junction x="133.858" y="41.148"/>
+</segment>
+</net>

Commit message: update
Parts:
- removed RRTC1: 10K, rcl:R-EU_R0805
- removed RTCINT: SOLDERJUMPERNO, _SparkFun:SOLDERJUMPERNO
Connections:
- removed net N$4: RRTC1.2, RTC.INT/SQW, RTCINT.1
- net D3: no longer RTCINT.2
- net VCC: no longer RRTC1.1
Changed lines of the file:
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@@
 <part name="RTC" library="_lh-library" deviceset="DS3231" device="" value="DS3231"/>
 <part name="BAT" library="SparkFunNew" deviceset="BATTERY" device="BATTERY_12MM_SMT" value="CR1220"/>
-<part name="RRTC1" library="rcl" deviceset="R-EU_" device="R0805" value="10K"/>
 <part name="P+9" library="supply1" deviceset="VCC" device=""/>
-<part name="RTCINT" library="_SparkFun" deviceset="SOLDERJUMPER" device="NO"/>
 <part name="X3" library="SparkFun" deviceset="RESONATOR" device="SMD" value="16 MHz"/>
 <part name="REMOTE" library="zetex" deviceset="PMOSSOT23" device="" value="FDN340P"/>
@@
 <attribute name="VALUE" x="13.97" y="151.892" size="1.778" layer="96"/>
 </instance>
-<instance part="RRTC1" gate="G$1" x="-45.466" y="168.148" smashed="yes" rot="R180">
-<attribute name="NAME" x="-48.006" y="166.878" size="1.778" layer="95" rot="R270"/>
-<attribute name="VALUE" x="-44.958" y="165.608" size="1.778" layer="96" rot="R270"/>
-</instance>
 <instance part="P+9" gate="VCC" x="-33.02" y="173.99"/>
-<instance part="RTCINT" gate="1" x="-55.88" y="162.306" smashed="yes" rot="R180">
-<attribute name="NAME" x="-53.34" y="166.116" size="1.778" layer="95" rot="R180"/>
-</instance>
 <instance part="X3" gate="G$1" x="10.16" y="41.91" rot="R270"/>
 <instance part="REMOTE" gate="A" x="140.462" y="41.148" rot="MR270"/>
@@
 <wire x1="-29.21" y1="163.83" x2="-40.386" y2="168.148" width="0.1524" layer="91"/>
 <wire x1="-40.386" y1="168.148" x2="-33.02" y2="171.45" width="0.1524" layer="91"/>
-<pinref part="RRTC1" gate="G$1" pin="1"/>
-<junction x="-40.386" y="168.148"/>
 <pinref part="RTC" gate="G$1" pin="VCC"/>
 </segment>
@@
 <wire x1="69.85" y1="31.75" x2="62.23" y2="31.75" width="0.1524" layer="91"/>
 <label x="66.04" y="31.75" size="1.778" layer="95"/>
-</segment>
-<segment>
-<pinref part="RTCINT" gate="1" pin="2"/>
-<wire x1="-60.96" y1="162.306" x2="-62.484" y2="167.132" width="0.1524" layer="91"/>
-<label x="-64.008" y="167.64" size="1.778" layer="95"/>
 </segment>
 </net>
@@
 </segment>
 </net>
-<net name="N$4" class="0">
-<segment>
-<pinref part="RRTC1" gate="G$1" pin="2"/>
-<pinref part="RTCINT" gate="1" pin="1"/>
-<wire x1="-50.8" y1="162.306" x2="-50.546" y2="168.148" width="0.1524" layer="91"/>
-<pinref part="RTC" gate="G$1" pin="INT/SQW"/>
-<wire x1="-50.8" y1="162.306" x2="-29.21" y2="162.306" width="0.1524" layer="91"/>
-<wire x1="-29.21" y1="162.306" x2="-29.21" y2="161.29" width="0.1524" layer="91"/>
-<junction x="-50.8" y="162.306"/>
-</segment>
-</net>

Commit message: update
Parts:
- added C9: .1uF, rcl:C-EUC0805
- added JP1: (no value), pinhead:PINHD-1X2
- added RM1, RM2: 10K, rcl:R-EU_R0805
Connections:
- new net VIN: RM1.2
- net A3: now also C9.2, RM1.1, RM2.2
- net GND: now also C9.1, RM2.1
Other:
- note added: "can add high side swith if drains too much power"
Changed lines of the file:
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@@
 <clearance class="0" value="0.2032"/>
 </class>
-<class number="1" name="power" width="0.381" drill="0">
+<class number="1" name="power" width="0.381" drill="0.3302">
 <clearance class="1" value="0.254"/>
 </class>
@@
 <part name="C8" library="resistor" deviceset="C-EU" device="C0805" value=".1u"/>
 <part name="JP4" library="SparkFun-Connectors" deviceset="M07" device=""/>
+<part name="JP1" library="pinhead" deviceset="PINHD-1X2" device=""/>
+<part name="GND4" library="supply1" deviceset="GND" device=""/>
+<part name="C9" library="rcl" deviceset="C-EU" device="C0805" value=".1uF"/>
+<part name="RM1" library="rcl" deviceset="R-EU_" device="R0805" value="10K"/>
+<part name="RM2" library="rcl" deviceset="R-EU_" device="R0805" value="10K"/>
 </parts>
 <sheets>
@@
 <plain>
 <text x="-113.284" y="94.996" size="1.778" layer="91">i2c pullups</text>
+<text x="44.196" y="181.61" size="1.778" layer="91">can add high side swith
+if drains too much power</text>
 </plain>
 <instances>
@@
 </instance>
 <instance part="JP4" gate="G$1" x="162.56" y="18.034" rot="R180"/>
+<instance part="JP1" gate="G$1" x="-58.42" y="139.7"/>
+<instance part="GND4" gate="1" x="87.884" y="147.828"/>
+<instance part="C9" gate="G$1" x="80.264" y="159.258" smashed="yes" rot="R180">
+<attribute name="NAME" x="82.423" y="156.972" size="1.778" layer="95" rot="R90"/>
+<attribute name="VALUE" x="84.963" y="156.972" size="1.778" layer="96" rot="R90"/>
+</instance>
+<instance part="RM1" gate="G$1" x="87.884" y="178.816" smashed="yes" rot="R90">
+<attribute name="NAME" x="86.614" y="181.356" size="1.778" layer="95" rot="R180"/>
+<attribute name="VALUE" x="85.344" y="177.038" size="1.778" layer="96" rot="R180"/>
+</instance>
+<instance part="RM2" gate="G$1" x="87.884" y="161.798" smashed="yes" rot="R90">
+<attribute name="NAME" x="86.614" y="164.338" size="1.778" layer="95" rot="R180"/>
+<attribute name="VALUE" x="85.344" y="160.02" size="1.778" layer="96" rot="R180"/>
+</instance>
 </instances>
 <busses>
@@
 <pinref part="JP4" gate="G$1" pin="1"/>
 </segment>
+<segment>
+<pinref part="GND4" gate="1" pin="GND"/>
+<wire x1="87.884" y1="150.368" x2="87.884" y2="152.654" width="0.1524" layer="91"/>
+<pinref part="C9" gate="G$1" pin="1"/>
+<wire x1="87.884" y1="152.654" x2="87.884" y2="156.718" width="0.1524" layer="91"/>
+<wire x1="80.264" y1="156.718" x2="80.264" y2="152.654" width="0.1524" layer="91"/>
+<wire x1="80.264" y1="152.654" x2="87.884" y2="152.654" width="0.1524" layer="91"/>
+<junction x="87.884" y="152.654"/>
+<pinref part="RM2" gate="G$1" pin="1"/>
+</segment>
 </net>
 <net name="VBUS" class="1">
@@
 <label x="66.04" y="54.61" size="1.778" layer="95"/>
 </segment>
+<segment>
+<wire x1="87.884" y1="166.878" x2="88.138" y2="169.164" width="0.1524" layer="91"/>
+<wire x1="88.138" y1="169.164" x2="87.884" y2="173.736" width="0.1524" layer="91"/>
+<wire x1="88.138" y1="169.164" x2="98.044" y2="168.91" width="0.1524" layer="91"/>
+<wire x1="98.044" y1="168.91" x2="97.282" y2="169.418" width="0.1524" layer="91"/>
+<label x="98.044" y="169.164" size="1.778" layer="95"/>
+<junction x="88.138" y="169.164"/>
+<pinref part="C9" gate="G$1" pin="2"/>
+<wire x1="88.138" y1="169.164" x2="80.264" y2="169.164" width="0.1524" layer="91"/>
+<wire x1="80.264" y1="169.164" x2="80.264" y2="164.338" width="0.1524" layer="91"/>
+<pinref part="RM1" gate="G$1" pin="1"/>
+<pinref part="RM2" gate="G$1" pin="2"/>
+</segment>
 </net>
 <net name="A5" class="0">
@@
 </segment>
 </net>
+<net name="VIN" class="1">
+<segment>
+<wire x1="87.884" y1="186.944" x2="87.884" y2="183.896" width="0.1524" layer="91"/>
+<label x="90.17" y="187.706" size="1.778" layer="95"/>
+<pinref part="RM1" gate="G$1" pin="2"/>
+</segment>
+</net>
 </nets>
 </sheet>
@@
 </schematic>
 </drawing>
+<compatibility>
+<note version="6.3" minversion="6.2.2" severity="warning">
+Since Version 6.2.2 text objects can contain more than one line,
+which will not be processed correctly with this version.
+</note>
+</compatibility>
 </eagle>
