File: hardware/riffle-0.4lp.sch (EAGLE design)
At the start: 41 parts, among them IC1 ATMEGA328P, IC2 MCP73831, IC3 CH340G, IC4 MCP1700-33, IC5 24AA128SN, IC6 MCP1700-33, J1 AYZ0202, X1 USBSMD, X2 12MHz, X3 16 MHz

Commit message: update
Parts:
- removed C9: .1uF, rcl:C-EUC0805
- added C12: .1u, resistor:C-EUC0805
- added REMOTE1: FDN340P, zetex:PMOSSOT23
- added RSD1, RSD2: 10K, adafruit2013:R-US_R0603
- added U1: RFM69W, ChipsParts:RFM69W
Connections:
- removed net VIN: RM1.2
- new net N$12: U1.ANT
- new net N$14: U1.GND@2
- new net N$15: C12.2, REMOTE1.D, RM1.2
- new net N$16: RSD1.2, U$1.DAT1
- new net N$17: RSD1.1, RSD2.2, U$1.VDD
- new net N$18: RSD2.1, U$1.DAT2
- new net N$19: U$1.CD/DAT3
- new net N$20: U$1.CMD
- new net N$21: U$1.CLK
- new net N$22: U$1.DAT0
- net A1: no longer JP4.3
- net A3: no longer C9.2
- net D10: now also REMOTE1.G
- net D3: now also JP4.3
- net D4: no longer REMOTE.G
- net D8: now also REMOTE.G
- net GND: now also C12.1, U$1.GND, U$1.GND1, U$1.GND2, U$1.GND3, U$1.GND4, U$1.SW_A, U$1.SW_B; no longer C9.1
- net VBAT: now also REMOTE1.S
Other:
- note removed: "can add high side swith if drains too much power"
- moved on the sheet: JP1, RM1

Commit message: update
Parts:
- removed C7: 0.1u, adafruit:C-USC0805K
- removed RN1: (no value), resistor-dil:4R-NEXB38V
- removed RSD: 10K, adafruit2013:R-US_R0603
- removed U1: RFM69W, ChipsParts:RFM69W
- added C9: .1u, resistor:C-EUC0805
- added JP3: (no value), SparkFun:M04SMD
- added RC1, RC2: 10K, adafruit2013:R-US_R0805
- added SDPWER: FDN340P, zetex:PMOSSOT23
- added STAT: 0805, led:LEDCHIPLED_0805
- C11: value 10u -> .1u
- C6: value 0.1u -> .1u; device adafruit:C-USC0805K -> adafruit2013:C-USC0805K
- JP2: device SparkFun-Connectors:M08 -> SparkFun:M04SMD
- RSD1, RSD2: value 10K -> 50k; device adafruit2013:R-US_R0603 -> adafruit2013:R-US_R0805
- renumbered REMOTE1 to BATTPOWER
Connections:
- removed net D10_SS: U$5.SEL
- removed net D11_MOSI: U$5.MOSI
- removed net D12_MISO: U$5.MISO
- removed net D13_SCK: U$5.SCK
- removed net N$10: CHG.A, RN1D.1
- removed net N$12: U1.ANT
- removed net N$14: U1.GND@2
- removed net N$19: U$1.CD/DAT3
- removed net N$20: U$1.CMD
- removed net N$21: U$1.CLK
- removed net N$22: U$1.DAT0
- net D2: no longer U$5.DIO0
- net D5: now also SDPWER.G
- net D7: now also U$1.CD/DAT3
- net D9: now also RC2.2
- net GND: now also C10.2, C11.1, C9.1, JP1.1, STAT.C; no longer C6.2
- net MISO: now also U$1.DAT0, U$5.MISO
- net MOSI: now also U$1.CMD, U$5.MOSI
- net N$17: now also RC2.1, STAT.A; no longer RSD1.1, RSD2.2, U$1.VDD
- net N$4: now also C9.2, RSD1.1, RSD2.2, SDPWER.D, U$1.VDD; no longer C6.1, IC3.V3, IC3.VCC
- net N$8: now also C11.2, IC3.V3, IC3.VCC; no longer C11.1
- net N$9: now also CHG.A, RC1.1; no longer C10.1, IC6.IN
- net RESET: now also C6.1; no longer C7.1
- net RST: now also C6.2; no longer C7.2
- net SCK: now also U$1.CLK, U$5.SCK
- net VBAT: now also JP1.2
- net VBUS: now also C10.1, IC6.IN, RC1.2; no longer C10.2, RN1D.2
- net VCC: now also SDPWER.S; no longer RSD.2
Other:
- moved on the sheet: C10, C11, C6
