File: hardware/riffle-0.4lp.brd (EAGLE design)
At the start: 102.7 x 18 mm, 41 parts, among them IC1 ATMEGA328P, IC2 MCP73831, IC3 CH340G, IC4 MCP1700-33, IC5 24AA128SN, IC6 MCP1700-33, J1 AYZ0202, X1 USBSMD, X2 12MHz, X3 16 MHz

Commit message: update
Parts:
- removed C9: .1uF, rcl:C0805@1
- added C12: .1u, resistor:C0805
- added REMOTE1: FDN340P, zetex:SOT-23
- added RSD1, RSD2: 10K, adafruit2013:R0603
- added U1: RFM69W, ChipsParts:RFM69W
- moved U$5 0.73 mm to (82.8, 16.1)
Connections:
- removed net VIN: RM1.2
- new net N$12: U1.10
- new net N$14: U1.11
- new net N$15: C12.2, REMOTE1.1, RM1.2
- new net N$16: RSD1.2, U$1.DAT1
- new net N$17: RSD1.1, RSD2.2, U$1.VDD
- new net N$18: RSD2.1, U$1.DAT2
- new net N$19: U$1.CD/DAT3
- new net N$20: U$1.CMD
- new net N$21: U$1.CLK
- new net N$22: U$1.DAT0
- net A1: no longer JP4.3
- net A3: no longer C9.2
- net D10: now also REMOTE1.3
- net D3: now also JP4.3
- net D4: no longer REMOTE.3
- net D8: now also REMOTE.3
- net GND: now also C12.1, U$1.GND1, U$1.GND2, U$1.GND3, U$1.GND4, U$1.SW_A, U$1.SW_B, U$1.VSS; no longer C9.1
- net VBAT: now also REMOTE1.2

Commit message: update
Parts:
- removed C7: 0.1u, adafruit:C0805K
- removed REMOTE1: FDN340P, zetex:SOT-23
- removed RN1: (no value), resistor-dil:EXB38V
- removed RSD: 10K, adafruit2013:R0603
- removed U1: RFM69W, ChipsParts:RFM69W
- added BATTPOWER, SDPWER: FDN340P, zetex:SOT-23
- added C9: .1u, resistor:C0805
- added JP3: (no value), SparkFun:1X04-SMD
- added RC1, RC2: 10K, adafruit2013:R0805
- added STAT: 0805, led:CHIPLED_0805
- C11: value 10u -> .1u
- C6: value 0.1u -> .1u; device adafruit:C0805K -> adafruit2013:C0805K
- JP2: device SparkFun-Connectors:1X08_ROUND -> SparkFun:1X04-SMD
- RSD1, RSD2: value 10K -> 50k; device adafruit2013:R0603 -> adafruit2013:R0805
- moved RSD2 98.9 mm to (82.7, 9.30), turned to 270 degrees
- moved C12 94.5 mm to (81.1, 15.1), turned to 90 degrees
- moved RSD1 94.5 mm to (80.8, 9.30), turned to 270 degrees
- moved U$5 66.2 mm to (16.6, 16.4)
- moved C4 65.0 mm to (81.1, 23.1), turned to 270 degrees
- moved RM1 63.4 mm to (75.1, 23.2), turned to 90 degrees
- moved RM2 62.3 mm to (78.0, 23.2), turned to 90 degrees
- moved JP2 56.7 mm to (29.2, 33.6), flipped to the bottom, turned to 270 degrees
- moved U$3 50.1 mm to (2.60, 17.8)
- moved I2C2 49.2 mm to (60.9, 23.9)
- moved I2C1 42.9 mm to (60.9, 21.9)
- moved C6 38.7 mm to (24.1, 8.80), turned to 180 degrees
- moved RC 36.2 mm to (15.9, 9.30)
- moved CHG 31.8 mm to (12.0, 8.80), turned to 90 degrees
- moved C5 26.8 mm to (45.1, 24.2), turned to 180 degrees
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Connections:
- removed net D10_SS: U$5.NSS
- removed net D11_MOSI: U$5.MOSI
- removed net D12_MISO: U$5.MISO
- removed net D13_SCK: U$5.SCK
- removed net N$10: CHG.A, RN1.4
- removed net N$12: U1.10
- removed net N$14: U1.11
- removed net N$19: U$1.CD/DAT3
- removed net N$20: U$1.CMD
- removed net N$21: U$1.CLK
- removed net N$22: U$1.DAT0
- net D10: now also BATTPOWER.3; no longer REMOTE1.3
- net D2: no longer U$5.DIO0
- net D5: now also SDPWER.3
- net D7: now also U$1.CD/DAT3
- net D9: now also RC2.2
- net GND: now also C10.2, C11.1, C9.1, JP1.1, STAT.C; no longer C6.2
- net MISO: now also U$1.DAT0, U$5.MISO
- net MOSI: now also U$1.CMD, U$5.MOSI
- net N$15: now also BATTPOWER.1; no longer REMOTE1.1
- net N$17: now also RC2.1, STAT.A; no longer RSD1.1, RSD2.2, U$1.VDD
- net N$4: now also C9.2, RSD1.1, RSD2.2, SDPWER.1, U$1.VDD; no longer C6.1, IC3.16, IC3.4
- net N$8: now also C11.2, IC3.16, IC3.4; no longer C11.1
- net N$9: now also CHG.A, RC1.1; no longer C10.1, IC6.2
- net RESET: now also C6.1; no longer C7.1
- net RST: now also C6.2; no longer C7.2
- net SCK: now also U$1.CLK, U$5.SCK
- net VBAT: now also BATTPOWER.2, JP1.2; no longer REMOTE1.2
- net VBUS: now also C10.1, IC6.2, RC1.2; no longer C10.2, RN1.5
- net VCC: now also SDPWER.2; no longer RSD.2

Commit message: update
Parts:
- moved U$3 81.7 mm to (84.2, 22.3)
- moved U$5 64.6 mm to (78.0, 36.4)
- moved STAT 3.03 mm to (3.00, 17.8), turned to 270 degrees
- moved IC4 1.73 mm to (36.3, 10.2), turned to 180 degrees
- moved RRST 1.04 mm to (29.7, 16.6)
- moved X2 1.00 mm to (24.6, 16.3)
- moved C3 0.70 mm to (41.3, 8.70)
- moved RC 0.64 mm to (16.3, 8.80)
- moved CHG 0.45 mm to (12.4, 8.60)
- moved IC2 0.40 mm to (24.4, 12.4), turned to 180 degrees
- moved IC6 0.32 mm to (19.7, 12.0), turned to 180 degrees
- moved C6 0.20 mm to (24.3, 8.80)
- moved X3 0.14 mm to (40.5, 12.5)
