File: hardware/riffle-0.95.brd (EAGLE design)
At the start: 72 x 18 mm, 47 parts, among them IC1 ATMEGA328P, IC2 MCP73831, IC3 CH340G, IC4 MCP1700-33, IC5 24AA128SN, IC6 MCP1700-33, J1 AYZ0202, X2 12MHz, X3 16 MHz

Commit message: update
Parts:
- moved REMOTE 0.89 mm to (51.2, 11.7)
- renumbered RTC to RTC-DS3231
Routing:
- net N$7: track 30.6 -> 32.1 mm
- net VCC: track 112.7 -> 113.6 mm
- net D3: track 43.5 -> 42.6 mm
- net D8: track 16.7 -> 17.5 mm
- net N$4: track 16.8 -> 16.0 mm
- net N$16: track 19.8 -> 20.4 mm
Other:
- board text added: "+"
- board text added: "-"
- board text added: "328p"
- board text added: "3V3"
- board text added: "A0"
- board text added: "A1"
- board text added: "A2"
- board text added: "ACT"
- board text added: "CH340G"
- board text added: "CHG"
- board text added: "D10"
- board text added: "D2"
- board text added: "D3"
- board text added: "D4"
- board text added: "D5"
- board text added: "GND"
- board text added: "IC2"
- board text added: "MISO"
- board text added: "MOSI"
- board text added: "OFF"
- board text added: "ON"
- board text added: "RESET"
- board text added: "RIFFLE-328p ver 0.95"
- board text added: "RX"
- board text added: "SCK"
- board text added: "SCL"
- board text added: "SDA"
- board text added: "TX"
- board text added: "VBAT"
- board text added: "VBUS"
- board text added: "X2"
- board text added: "battpwr"
- board text added: "eeprom"
- board text added: "publiclab.org/wiki/riffle"
