File: hardware/riffle-0.95.sch (EAGLE design)
At the start: 47 parts, among them IC1 ATMEGA328P, IC2 MCP73831, IC3 CH340G, IC4 MCP1700-33, IC5 24AA128SN, IC6 MCP1700-33, J1 AYZ0202, X2 12MHz, X3 16 MHz

Commit message: update
Parts:
- renumbered RTC to RTC-DS3231
Changed lines of the file:
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@@
 <part name="P+5" library="supply1" deviceset="VCC" device=""/>
 <part name="P+10" library="supply1" deviceset="VCC" device=""/>
-<part name="RTC" library="_lh-library" deviceset="DS3231" device="" value="DS3231"/>
+<part name="RTC-DS3231" library="_lh-library" deviceset="DS3231" device="" value="DS3231"/>
 <part name="BAT" library="SparkFunNew" deviceset="BATTERY" device="BATTERY_12MM_SMT" value="CR1220"/>
 <part name="P+9" library="supply1" deviceset="VCC" device=""/>
@@
 <instance part="P+5" gate="VCC" x="42.926" y="164.338"/>
 <instance part="P+10" gate="VCC" x="53.086" y="165.354"/>
-<instance part="RTC" gate="G$1" x="-16.51" y="157.48"/>
+<instance part="RTC-DS3231" gate="G$1" x="-16.51" y="157.48"/>
 <instance part="BAT" gate="G$1" x="8.89" y="154.432" smashed="yes" rot="R270">
 <attribute name="NAME" x="13.97" y="154.432" size="1.778" layer="95"/>
@@
 <junction x="-31.75" y="151.13"/>
 <junction x="-31.75" y="148.59"/>
-<pinref part="RTC" gate="G$1" pin="GND"/>
-<pinref part="RTC" gate="G$1" pin="NC@8"/>
-<pinref part="RTC" gate="G$1" pin="NC@7"/>
-<pinref part="RTC" gate="G$1" pin="NC@6"/>
-<pinref part="RTC" gate="G$1" pin="NC@5"/>
-<pinref part="RTC" gate="G$1" pin="NC@1"/>
-<pinref part="RTC" gate="G$1" pin="NC@2"/>
-<pinref part="RTC" gate="G$1" pin="NC@3"/>
-<pinref part="RTC" gate="G$1" pin="NC@4"/>
+<pinref part="RTC-DS3231" gate="G$1" pin="GND"/>
+<pinref part="RTC-DS3231" gate="G$1" pin="NC@8"/>
+<pinref part="RTC-DS3231" gate="G$1" pin="NC@7"/>
+<pinref part="RTC-DS3231" gate="G$1" pin="NC@6"/>
+<pinref part="RTC-DS3231" gate="G$1" pin="NC@5"/>
+<pinref part="RTC-DS3231" gate="G$1" pin="NC@1"/>
+<pinref part="RTC-DS3231" gate="G$1" pin="NC@2"/>
+<pinref part="RTC-DS3231" gate="G$1" pin="NC@3"/>
+<pinref part="RTC-DS3231" gate="G$1" pin="NC@4"/>
 <pinref part="BAT" gate="G$1" pin="-"/>
 </segment>
@@
 <wire x1="-29.21" y1="163.83" x2="-37.592" y2="163.83" width="0.1524" layer="91"/>
 <wire x1="-37.592" y1="163.83" x2="-37.592" y2="171.45" width="0.1524" layer="91"/>
-<pinref part="RTC" gate="G$1" pin="VCC"/>
+<pinref part="RTC-DS3231" gate="G$1" pin="VCC"/>
 </segment>
 <segment>
@@
 <segment>
 <wire x1="-3.81" y1="163.83" x2="12.446" y2="163.83" width="0.1524" layer="91"/>
-<pinref part="RTC" gate="G$1" pin="SDA"/>
+<pinref part="RTC-DS3231" gate="G$1" pin="SDA"/>
 <label x="13.208" y="163.83" size="1.778" layer="95"/>
 </segment>
@@
 <segment>
 <wire x1="-3.81" y1="166.37" x2="12.446" y2="166.37" width="0.1524" layer="91"/>
-<pinref part="RTC" gate="G$1" pin="SCL"/>
+<pinref part="RTC-DS3231" gate="G$1" pin="SCL"/>
 <label x="12.954" y="166.878" size="1.778" layer="95"/>
 </segment>
@@
 <wire x1="-3.81" y1="161.29" x2="8.89" y2="161.29" width="0.1524" layer="91"/>
 <wire x1="8.89" y1="161.29" x2="8.89" y2="159.512" width="0.1524" layer="91"/>
-<pinref part="RTC" gate="G$1" pin="VBAT"/>
+<pinref part="RTC-DS3231" gate="G$1" pin="VBAT"/>
 <pinref part="BAT" gate="G$1" pin="+"/>
 </segment>
