File: hardware/riffle-0.96-tab.brd (EAGLE design)
At the start: 72 x 28 mm, 47 parts, among them IC1 ATMEGA328P, IC2 MCP73831, IC3 CH340G, IC4 MCP1700-33, IC5 24AA128SN, IC6 MCP1700-33, J1 AYZ0202, J2 USB MICRO, X2 12MHz, X3 16 MHz

Commit message: update
Parts:
- removed J2: USB MICRO, SmartPrj:CON2_USB_MICRO_B_AT
- added U$4: (no value), Testing:USB-AB-MICRO-SMD_V02_BOSS
Connections:
- net D+: now also U$4.D+1; no longer J2.P3
- net D-: now also U$4.D-1; no longer J2.P2
- net GND: now also U$4.GND1; no longer J2.P5, J2.S1, J2.S2, J2.S3, J2.S4, J2.S5, J2.S6
- net N$19: now also U$4.VBUS1; no longer J2.P1
Routing:
- net GND: track 254.7 -> 243.8 mm
Other:
- board size 72 x 28 mm -> 72 x 28.2 mm
