File: hardware/riffle-beta-0.1.0.sch (EAGLE design)
At the start: 48 parts, among them IC1 ATMEGA328P, IC2 MCP73831, IC3 CH340G, IC5 24AA128SN, IC7 MIC5225-3.3V, IC8 MIC5225-3.3V, J1 AYZ0202, X2 12MHz, X3 16 MHz

Commit message: update
Parts:
- added RTC: (no value), wirepad:SMD2
Connections:
- new net N$12: RTC-DS3231.INT/SQW, RTC.P
Other:
- moved on the sheet: C8, C9, IC5, ISP, JP3, JP5, R7, R8, REMOTE, SDPWER, U$1

Commit message: update
Parts:
- removed C6: 10uF, SparkFun:CAP0603-CAP
- removed IC7, IC8: MIC5225-3.3V, adafruit:LP298XS
- removed RTC: (no value), wirepad:SMD2
- added C13, C14: 10uF, SparkFun:CAP0603-CAP
- added IC4, IC6: MCP1700-33, adafruit:MCP1700SOT89
- R7, R8: value 50K -> 10K
Connections:
- removed net D5: IC1.PD5(T1), JP3.4
- removed net N$12: RTC-DS3231.INT/SQW, RTC.P
- new net D5/RST: JP3.4
- new net D5/RTC: IC1.PD5(T1), RTC-DS3231.INT/SQW
- net A1: now also JP5.12; no longer JP3.1
- net A2: now also JP5.10; no longer JP3.2
- net GND: now also C13.2, C14.2, IC4.GND, IC6.GND; no longer C6.2, IC7.GND, IC8.GND
- net N$8: now also IC6.OUT; no longer IC7.VOUT
- net RXD: now also JP3.2; no longer JP5.10
- net TXD: now also JP3.1; no longer JP5.12
- net VBUS: now also IC6.IN; no longer IC7.EN, IC7.VIN
- net VCC: now also C14.1, IC4.OUT; no longer C6.1, IC8.VOUT
- net VDD: now also C13.1, IC4.IN; no longer IC8.EN, IC8.VIN
Other:
- moved on the sheet: JP3

Commit message: update
Parts:
- removed D3, D4: SCHOTTKY, adafruit:DIODE_SOD-123FL
- removed L1: 500mA, adafruit:PTCFUSE-1206
Connections:
- removed net D5/RST: JP3.4
- removed net N$10: D3.A, L1.2
- removed net N$14: D4.A, JP1.2
- removed net N$19: J2.5V, L1.1
- new net VGEN: CN2.2, J1.6, JP1.2
- net D5/RTC: now also JP3.4
- net GND: now also CN2.1
- net VBAT: now also J1.4; no longer D4.C, J1.2
- net VBUS: now also J2.5V; no longer D3.C
- net VDD: now also J1.2; no longer J1.3
Other:
- moved on the sheet: CN1, CN2, IC6, J1, J2, JP1
