File: hardware/riffle-beta-0.1.0.brd (EAGLE design)
At the start: 102.6 x 18.2 mm, 48 parts, among them IC1 ATMEGA328P, IC2 MCP73831, IC3 CH340G, IC5 24AA128SN, IC7 MIC5225-3.3V, IC8 MIC5225-3.3V, J1 AYZ0202, X2 12MHz, X3 16 MHz

Commit message: update
Parts:
- added RTC: (no value), wirepad:SMD1,27-2,54
Connections:
- new net N$12: RTC-DS3231.3, RTC.1
Changed lines of the file:
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@@
 <element name="IC7" library="adafruit" package="SOT23-5L" value="MIC5225-3.3V" x="51.7144" y="15.113"/>
 <element name="IC8" library="adafruit" package="SOT23-5L" value="MIC5225-3.3V" x="55.0164" y="15.2146"/>
+<element name="RTC" library="wirepad" package="SMD1,27-2,54" value="" x="94.107" y="15.7734" rot="MR90"/>
 </elements>
 <signals>
@@
 <wire x1="18.3892" y1="4.7498" x2="18.4892" y2="2.0798" width="0" layer="19" extent="1-1"/>
 </signal>
+<signal name="N$12">
+<contactref element="RTC-DS3231" pad="3"/>
+<contactref element="RTC" pad="1"/>
+<wire x1="94.107" y1="15.7734" x2="50.2868" y2="7.2796" width="0" layer="19" extent="1-1"/>
+</signal>
 </signals>

Commit message: update
Parts:
- removed C6: 10uF, SparkFun:0603-CAP
- removed IC7, IC8: MIC5225-3.3V, adafruit:SOT23-5L
- removed RTC: (no value), wirepad:SMD1,27-2,54
- added C13, C14: 10uF, SparkFun:0603-CAP
- added IC4, IC6: MCP1700-33, adafruit:SOT89
- R7, R8: value 50K -> 10K
- moved L1 66.2 mm to (9.43, 7.88), turned to 180 degrees
- moved C4 44.2 mm to (18.8, 13.8), turned to 180 degrees
- moved C5 35.4 mm to (21.4, 4.07), turned to 180 degrees
- moved R5 24.9 mm to (61.1, 2.46)
- moved D1 24.5 mm to (13.8, 16.9), turned to 180 degrees
- moved R6 23.1 mm to (61.1, 1.22), turned to 180 degrees
- moved C2 21.9 mm to (10.1, 15.5), turned to 0 degrees
- moved J1 19.2 mm to (27.0, 14.1), turned to 0 degrees
- moved R7 19.1 mm to (96.5, 9.05)
- moved IC2 18.6 mm to (18.1, 16.3), turned to 90 degrees
- moved R9 18.5 mm to (33.4, 16.2)
- moved JP3 17.2 mm to (40.3, 9.00)
- moved C7 17.1 mm to (48.9, 1.17)
- moved R8 15.6 mm to (96.3, 15.5), turned to 270 degrees
- moved R10 15.4 mm to (48.5, 16.5)
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Connections:
- removed net D5: IC1.9, JP3.4
- removed net N$12: RTC-DS3231.3, RTC.1
- new net D5/RST: JP3.4
- new net D5/RTC: IC1.9, RTC-DS3231.3
- net A1: now also JP5.12; no longer JP3.1
- net A2: now also JP5.10; no longer JP3.2
- net GND: now also C13.2, C14.2, IC4.1, IC6.1; no longer C6.2, IC7.2, IC8.2
- net N$8: now also IC6.3; no longer IC7.5
- net RXD: now also JP3.2; no longer JP5.10
- net TXD: now also JP3.1; no longer JP5.12
- net VBUS: now also IC6.2; no longer IC7.1, IC7.3
- net VCC: now also C14.1, IC4.3; no longer C6.1, IC8.5
- net VDD: now also C13.1, IC4.2; no longer IC8.1, IC8.3
Routing:
- net GND: track 0.00 -> 296.5 mm, vias 0 -> 15
- net VBAT: track 0.00 -> 138.5 mm, vias 0 -> 9
- net VCC: track 0.00 -> 132.9 mm, vias 0 -> 10
- net VBUS: track 0.00 -> 112.2 mm, vias 0 -> 8
- net SCL: track 0.00 -> 96.2 mm, vias 0 -> 6
- net SDA: track 0.00 -> 86.0 mm, vias 0 -> 6
- net RXD: track 0.00 -> 64.9 mm, vias 0 -> 4
- net TXD: track 0.00 -> 57.8 mm, vias 0 -> 8
- net RESET: track 0.00 -> 54.4 mm, vias 0 -> 4
- net N$8: track 0.00 -> 51.8 mm, vias 0 -> 3
- net N$4: track 0.00 -> 42.8 mm, vias 0 -> 2
- net SCK: track 0.00 -> 41.5 mm, vias 0 -> 3
- net MISO: track 0.00 -> 40.4 mm, vias 0 -> 3
- net MOSI: track 0.00 -> 40.3 mm, vias 0 -> 2
- net A1: track 0.00 -> 36.9 mm, vias 0 -> 3
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Other:
- board size 102.6 x 18.2 mm -> 104.8 x 18 mm
- board text removed: "328p"
- board text removed: "ACT"
- board text removed: "CH340G"
- board text removed: "D5"
- board text removed: "GND"
- board text removed: "IC2"
- board text removed: "MISO"
- board text removed: "MOSI"
- board text removed: "OFF"
- board text removed: "ON"
- board text removed: "RIFFLE-328p ver 0.95"
- board text removed: "RST"
- board text removed: "SCK"
- board text removed: "VBUS"
- board text removed: "X2"
- board text removed: "all dimensions in mm"
- board text removed: "battpwr"
- board text removed: "eeprom"
- board text removed: "publiclab.org/wiki/riffle"

Commit message: update
Parts:
- removed D3, D4: SCHOTTKY, adafruit:SOD-123FL
- removed L1: 500mA, adafruit:R1206
- moved R9 15.4 mm to (48.8, 15.5)
- moved R2 13.4 mm to (10.6, 7.65), turned to 180 degrees
- moved D1 9.25 mm to (14.5, 7.72), turned to 0 degrees
- moved R1 6.31 mm to (16.2, 16.9), turned to 180 degrees
- moved C4 6.09 mm to (14.6, 9.37)
- moved C2 2.58 mm to (12.3, 16.9), turned to 180 degrees
- moved IC2 2.49 mm to (20.6, 15.9)
- moved C1 1.37 mm to (8.75, 16.9), turned to 0 degrees
- moved IC6 1.20 mm to (15.7, 13.3)
- moved C5 1.02 mm to (20.9, 4.94)
- moved JP1 0.65 mm to (10.5, 12.2), turned to 90 degrees
- moved C13 0.65 mm to (20.9, 3.17)
- moved R4 0.58 mm to (64.2, 4.50)
- moved R10 0.57 mm to (48.7, 17.0)
- moved C11 0.51 mm to (65.1, 1.36)
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Connections:
- removed net D5/RST: JP3.4
- removed net N$10: D3.A, L1.2
- removed net N$14: D4.A, JP1.2
- removed net N$19: J2.1, L1.1
- new net VGEN: CN2.1, J1.4, JP1.2
- net D5/RTC: now also JP3.4
- net GND: now also CN2.2
- net VBAT: now also J1.6; no longer D4.C, J1.2
- net VBUS: now also J2.1; no longer D3.C
- net VDD: now also J1.2; no longer J1.1
Routing:
- net VBUS: track 112.2 -> 80.5 mm, vias 8 -> 3
- net N$3: track 15.7 -> 38.6 mm
- net D5/RTC: track 35.1 -> 57.4 mm, vias 2 -> 5
- net VGEN: track 0.00 -> 21.0 mm, vias 0 -> 3
- net N$8: track 51.8 -> 31.5 mm, vias 3 -> 5
- net VCC: track 132.9 -> 113.4 mm, vias 10 -> 12
- net AREF: track 24.1 -> 39.4 mm
- net N$5: track 6.32 -> 16.2 mm
- net SCL: track 96.2 -> 88.2 mm, vias 6 -> 4
- net SLD: track 12.1 -> 20.1 mm
- net RXD: track 64.9 -> 57.9 mm
- net N$6: track 11.4 -> 18.0 mm
- net N$10: track 6.13 -> 0.00 mm
- net A2: track 31.6 -> 37.7 mm, vias 4 -> 1
- net D9: track 18.9 -> 24.7 mm
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Other:
- board text added: "3.7-6V"
- board text added: "D5/RTC"
- board text added: "GND"
- board text added: "Gen"
- board text added: "Lith"
- board text added: "RXD"
- board text added: "Riffle Beta 0.1.0"
- board text added: "TXD"
- board text added: "VBUS"
- board text removed: "3.7-12V"

Commit message: update
Parts:
- moved ISP 0.30 mm to (69.0, 15.2)
Routing:
- net AREF: track 39.4 -> 15.0 mm
- net SDA: track 86.3 -> 110.6 mm, vias 7 -> 5
- net N$15: track 24.7 -> 48.3 mm
- net VBUS: track 80.5 -> 99.2 mm, vias 3 -> 2
- net SCL: track 88.2 -> 74.4 mm, vias 4 -> 5
- net N$3: track 38.6 -> 24.8 mm, vias 2 -> 4
- net GND: track 299.8 -> 309.8 mm, vias 12 -> 14
- net VCC: track 113.4 -> 123.1 mm, vias 12 -> 11
- net VBAT: track 138.2 -> 128.9 mm, vias 4 -> 6
- net N$4: track 38.5 -> 30.7 mm
- net MOSI: track 39.8 -> 47.4 mm, vias 4 -> 2
- net D2: track 27.4 -> 33.4 mm
- net D7: track 13.2 -> 7.78 mm, vias 2 -> 0
- net D3: track 26.7 -> 31.9 mm, vias 2 -> 1
- net N$6: track 18.0 -> 12.9 mm
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Other:
- board text added: "Lith/USB"
- board text removed: "Lith"
