File: hardware/riffle-beta-0.1.0/riffle-beta-0.1.3.1.sch (EAGLE design)
At the start: 46 parts, among them IC1 ATMEGA328P, IC3 CH340G, IC4 MCP1700-33, IC5 24AA128SN, IC6 MCP1700-33, J1 AYZ0202, U1 MCP73831T-2ACI/OT, X2 12MHz, X3 16 MHz

Commit message: update
Connections:
- net GND: now also JP1.2; no longer JP1.1
- net VGEN: now also JP1.1; no longer JP1.2
Other:
- moved on the sheet: JP1
Changed lines of the file:
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@@
 <instance part="GND1" gate="1" x="134.62" y="29.21" rot="R270"/>
 <instance part="P+6" gate="VCC" x="166.878" y="31.75"/>
-<instance part="JP1" gate="G$1" x="-80.264" y="82.55"/>
+<instance part="JP1" gate="G$1" x="-91.44" y="83.82" rot="R180"/>
 <instance part="GND4" gate="1" x="88.392" y="147.828"/>
 <instance part="U$1" gate="G$1" x="206.502" y="87.122"/>
@@
 </segment>
 <segment>
-<pinref part="JP1" gate="G$1" pin="1"/>
-<wire x1="-82.804" y1="85.09" x2="-92.202" y2="85.09" width="0.1524" layer="91"/>
-<wire x1="-92.202" y1="85.09" x2="-92.202" y2="85.344" width="0.1524" layer="91"/>
-<label x="-96.52" y="85.09" size="1.778" layer="95"/>
+<wire x1="-78.74" y1="83.82" x2="-88.9" y2="83.82" width="0.1524" layer="91"/>
+<label x="-78.74" y="83.82" size="1.778" layer="95"/>
+<pinref part="JP1" gate="G$1" pin="2"/>
 </segment>
 <segment>
@@
 </segment>
 <segment>
-<wire x1="-82.804" y1="82.55" x2="-94.234" y2="82.55" width="0.1524" layer="91"/>
-<wire x1="-94.234" y1="82.55" x2="-94.234" y2="83.058" width="0.1524" layer="91"/>
-<label x="-96.012" y="82.804" size="1.778" layer="95"/>
-<pinref part="JP1" gate="G$1" pin="2"/>
-</segment>
-<segment>
+<wire x1="-88.9" y1="81.28" x2="-78.74" y2="81.28" width="0.1524" layer="91"/>
+<label x="-78.74" y="81.28" size="1.778" layer="95"/>
+<pinref part="JP1" gate="G$1" pin="1"/>
+</segment>
+<segment>
