File: hardware/riffle-beta-0.1.0/riffle-beta-0.1.5.sch (EAGLE design)
At the start: 51 parts, among them IC1 ATMEGA328P, IC3 CH340G, IC4 MCP1700-33, IC5 24AA128SN, IC6 MCP1700-33, J1 AYZ0202, Q1 FDN340P, U1 MCP73831T-2ACI/OT, X2 12MHz, X3 16 MHz

Commit message: update
Parts:
- D3: value SCHOTTKY -> SCHOTTKY SM4002PL-TP
Changed lines of the file:
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@@
 <part name="J1" library="SparkFunNew" deviceset="AYZ0202" device=""/>
 <part name="Q1" library="zetex" deviceset="PMOSSOT23" device="" value="FDN340P"/>
-<part name="D3" library="adafruit" deviceset="DIODE" device="_SOD-123FL" value="SCHOTTKY"/>
+<part name="D3" library="adafruit" deviceset="DIODE" device="_SOD-123FL" value="SCHOTTKY SM4002PL-TP"/>
 <part name="C5" library="SparkFun" deviceset="CAP" device="0603-CAP" value="1uF"/>
 <part name="C6" library="SparkFun" deviceset="CAP" device="0603-CAP" value="10uF"/>
@@
 <text x="-91.44" y="127" size="3.81" layer="91">USB-SERIAL</text>
 <text x="20.32" y="50.8" size="3.81" layer="91">Atmel328p</text>
-<text x="7.62" y="154.94" size="3.81" layer="91">Power Management</text>
+<text x="-7.62" y="167.64" size="3.81" layer="91">Power Management</text>
 <text x="-17.78" y="228.6" size="3.81" layer="91">RTC</text>
 <text x="231.14" y="233.68" size="3.81" layer="91">uSD</text>
@@
 </instance>
 <instance part="Q1" gate="A" x="134.62" y="124.46" rot="MR270"/>
-<instance part="D3" gate="G$1" x="149.86" y="137.16" rot="R270"/>
+<instance part="D3" gate="G$1" x="149.86" y="137.16" smashed="yes" rot="R270">
+<attribute name="NAME" x="152.4" y="139.7" size="1.27" layer="95" rot="R270"/>
+<attribute name="VALUE" x="146.05" y="149.86" size="1.27" layer="96" rot="R270"/>
+</instance>
 <instance part="C5" gate="G$1" x="149.86" y="111.76" smashed="yes">
 <attribute name="NAME" x="146.304" y="109.093" size="1.778" layer="95" rot="R180"/>
-<attribute name="VALUE" x="148.844" y="115.951" size="1.778" layer="96" rot="R180"/>
+<attribute name="VALUE" x="146.304" y="115.951" size="1.778" layer="96" rot="R180"/>
 </instance>
 <instance part="C6" gate="G$1" x="93.98" y="114.3" smashed="yes">

Commit message: update
Parts:
- D3: value SCHOTTKY SM4002PL-TP -> SCHOTTKY MBR120VLSFT3G
Changed lines of the file:
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@@
 <part name="J1" library="SparkFunNew" deviceset="AYZ0202" device=""/>
 <part name="Q1" library="zetex" deviceset="PMOSSOT23" device="" value="FDN340P"/>
-<part name="D3" library="adafruit" deviceset="DIODE" device="_SOD-123FL" value="SCHOTTKY SM4002PL-TP"/>
+<part name="D3" library="adafruit" deviceset="DIODE" device="_SOD-123FL" value="SCHOTTKY MBR120VLSFT3G"/>
 <part name="C5" library="SparkFun" deviceset="CAP" device="0603-CAP" value="1uF"/>
 <part name="C6" library="SparkFun" deviceset="CAP" device="0603-CAP" value="10uF"/>
@@
 <instance part="D3" gate="G$1" x="149.86" y="137.16" smashed="yes" rot="R270">
 <attribute name="NAME" x="152.4" y="139.7" size="1.27" layer="95" rot="R270"/>
-<attribute name="VALUE" x="146.05" y="149.86" size="1.27" layer="96" rot="R270"/>
+<attribute name="VALUE" x="146.05" y="144.78" size="1.27" layer="96" rot="R270"/>
 </instance>
 <instance part="C5" gate="G$1" x="149.86" y="111.76" smashed="yes">
