File: hardware/riffle-beta-0.1.0/riffle-beta-0.1.5.brd (EAGLE design)
At the start: 104.8 x 18 mm, 51 parts, among them IC1 ATMEGA328P, IC3 CH340G, IC4 MCP1700-33, IC5 24AA128SN, IC6 MCP1700-33, J1 AYZ0202, Q1 FDN340P, U1 MCP73831T-2ACI/OT, X2 12MHz, X3 16 MHz

Commit message: update
Parts:
- D3: value SCHOTTKY -> SCHOTTKY SM4002PL-TP
Changed lines of the file:
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@@
 <attribute name="OC_FARNELL" value="unknown" x="-0.2286" y="-6.477" size="1.778" layer="27" display="off"/>
 </element>
-<element name="D3" library="adafruit" package="SOD-123FL" value="SCHOTTKY" x="0.0508" y="-9.5758"/>
+<element name="D3" library="adafruit" package="SOD-123FL" value="SCHOTTKY SM4002PL-TP" x="0.0508" y="-9.5758"/>
 <element name="C5" library="SparkFun" package="0603-CAP" value="1uF" x="-0.6096" y="-12.6746"/>
 <element name="C6" library="SparkFun" package="0603-CAP" value="10uF" x="-0.6096" y="-15.6464"/>

Commit message: update
Parts:
- D3: value SCHOTTKY SM4002PL-TP -> SCHOTTKY MBR120VLSFT3G
Changed lines of the file:
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@@
 <attribute name="OC_FARNELL" value="unknown" x="-0.2286" y="-6.477" size="1.778" layer="27" display="off"/>
 </element>
-<element name="D3" library="adafruit" package="SOD-123FL" value="SCHOTTKY SM4002PL-TP" x="0.0508" y="-9.5758"/>
+<element name="D3" library="adafruit" package="SOD-123FL" value="SCHOTTKY MBR120VLSFT3G" x="0.0508" y="-9.5758"/>
 <element name="C5" library="SparkFun" package="0603-CAP" value="1uF" x="-0.6096" y="-12.6746"/>
 <element name="C6" library="SparkFun" package="0603-CAP" value="10uF" x="-0.6096" y="-15.6464"/>
