File: hardware/riffle-beta-0.1.0/riffle-beta-0.1.7.brd (EAGLE design)
At the start: 104.8 x 18 mm, 56 parts, among them IC1 ATMEGA328P, IC3 CH340G, IC4 MCP1700-33, IC5 24AA128SN, IC6 MCP1700-33, J1 AYZ0202, U1 MCP73831T-2ACI/OT, X2 12MHz, X3 16 MHz

Commit message: update
Parts:
- moved C3 27.1 mm to (67.7, 2.30)
- moved R3 18.4 mm to (67.8, 3.78), turned to 0 degrees
- moved SJ4 14.0 mm to (42.3, 1.42)
- moved SJ3 14.0 mm to (39.2, 1.40)
- moved SJ5 14.0 mm to (45.3, 1.50)
- moved C10 12.6 mm to (81.3, 1.16)
- moved C11 12.0 mm to (77.1, 1.13)
- moved D2 2.51 mm to (67.8, 0.94)
- moved C7 1.27 mm to (49.7, 2.03), turned to 90 degrees
- moved C14 0.43 mm to (37.6, 1.70), turned to 180 degrees
- moved IC3 0.22 mm to (27.3, 5.24)
- moved C6 0.20 mm to (21.8, 1.04)
- moved IC4 0.19 mm to (33.4, 2.57)
- moved D5 0.18 mm to (21.3, 2.87)
- moved D4 0.13 mm to (21.3, 4.95)
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