File: hardware/riffle-beta-0.1.0/riffle-beta-0.1.7.1.brd (EAGLE design)
At the start: 104.8 x 18 mm, 54 parts, among them IC1 ATMEGA328P, IC3 CH340G, IC4 MCP1700-33, IC5 24AA128SN, IC6 MCP1700-33, J1 AYZ0202, U1 MCP73831T-2ACI/OT, X2 12MHz, X3 16 MHz

Commit message: update
Parts:
- moved C14 2.17 mm to (39.8, 1.45)
- moved SJ3 1.55 mm to (43.5, 1.60)
Routing:
- net VDD: track 71.7 -> 78.4 mm
- net N$20: track 29.2 -> 32.0 mm
- net GND: track 308.2 -> 309.5 mm
Other:
- board text added: "T1"
