File: hardware/riffle-beta-0.1.0/riffle-beta-0.1.8.brd (EAGLE design)
At the start: 104.8 x 18 mm, 51 parts, among them IC1 ATMEGA328P, IC3 CH340G, IC4 MCP1700-33, IC5 24AA128SN, IC6 MCP1700-33, J1 AYZ0202, U1 MCP73831T-2ACI/OT, X2 12MHz, X3 16 MHz

Commit message: update
Parts:
- moved C3 25.8 mm to (42.0, 1.61), turned to 180 degrees
- moved C14 0.16 mm to (37.8, 1.57)
Connections:
- removed net N$14: C13.1, IC4.2, J1.2
- new net VIN: BATTPOWER.2, C13.1, IC4.2, J1.2
- net VBAT: no longer BATTPOWER.2
Routing:
- net VIN: track 0.00 -> 62.4 mm, vias 0 -> 3
- net RST: track 72.4 -> 18.2 mm, vias 2 -> 0
- net RESET: track 28.2 -> 65.3 mm, vias 3 -> 6
- net VCC: track 138.8 -> 105.9 mm, vias 8 -> 9
- net GND: track 318.8 -> 297.2 mm, vias 16 -> 9
- net SCL: track 104.5 -> 84.7 mm, vias 5 -> 8
- net N$14: track 19.8 -> 0.00 mm
- net A0: track 47.0 -> 30.7 mm
- net RXD: track 52.8 -> 68.6 mm, vias 2 -> 4
- net N$2: track 31.5 -> 15.8 mm
- net A2: track 32.5 -> 44.9 mm
- net N$10: track 24.2 -> 36.6 mm, vias 1 -> 2
- net D2: track 27.8 -> 39.6 mm, vias 3 -> 2
- net N$15: track 18.9 -> 29.6 mm, vias 2 -> 4
- net SLD: track 9.49 -> 18.4 mm, vias 0 -> 2
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