File: hardware/riffle-beta-0.1.0/riffle-beta-0.1.8.sch (EAGLE design)
At the start: 51 parts, among them IC1 ATMEGA328P, IC3 CH340G, IC4 MCP1700-33, IC5 24AA128SN, IC6 MCP1700-33, J1 AYZ0202, U1 MCP73831T-2ACI/OT, X2 12MHz, X3 16 MHz

Commit message: update
Connections:
- removed net N$14: C13.1, IC4.IN, J1.2
- new net VIN: BATTPOWER.S, C13.1, IC4.IN, J1.2
- net VBAT: no longer BATTPOWER.S
Changed lines of the file:
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@@
-</segment>
-<segment>
-<pinref part="BATTPOWER" gate="A" pin="S"/>
-<wire x1="331.216" y1="279.908" x2="338.328" y2="279.908" width="0.1524" layer="91"/>
-<wire x1="338.328" y1="279.908" x2="338.328" y2="282.448" width="0.1524" layer="91"/>
-<label x="338.074" y="283.718" size="1.778" layer="95"/>
 </segment>
 <segment>
@@
 </segment>
 </net>
-<net name="N$14" class="0">
+<net name="VIN" class="0">
 <segment>
 <pinref part="IC4" gate="1" pin="IN"/>
@@
 <wire x1="220.98" y1="127" x2="246.38" y2="127" width="0.1524" layer="91"/>
 <junction x="246.38" y="127"/>
-</segment>
-</net>
+<label x="231.14" y="129.54" size="1.778" layer="95"/>
+</segment>
+<segment>
+<pinref part="BATTPOWER" gate="A" pin="S"/>
+<wire x1="331.216" y1="279.908" x2="338.328" y2="279.908" width="0.1524" layer="91"/>
+<wire x1="338.328" y1="279.908" x2="338.328" y2="282.448" width="0.1524" layer="91"/>
+<label x="338.074" y="283.718" size="1.778" layer="95"/>
+</segment>
+</net>
