File: hardware/riffle-beta-0.1.0/riffle-beta-0.1.8.5.brd (EAGLE design)
At the start: 104.8 x 18 mm, 51 parts, among them IC1 ATMEGA328P, IC3 CH340G, IC4 MCP1700-33, IC5 24AA128SN, IC6 MCP1700-33, J1 AYZ0202, U1 MCP73831T-2ACI/OT, X2 12MHz, X3 16 MHz

Commit message: update
Parts:
- C2: value 0.1uF -> 10uF
Changed lines of the file:
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@@
 <attribute name="VALUE" x="7.049" y="15.774" size="0.4064" layer="27" font="vector"/>
 </element>
-<element name="C2" library="SparkFun" package="0603-CAP" value="0.1uF" x="11.3448" y="16.8882" smashed="yes" rot="R180">
+<element name="C2" library="SparkFun" package="0603-CAP" value="10uF" x="11.3448" y="16.8882" smashed="yes" rot="R180">
 <attribute name="NAME" x="11.6623" y="16.0627" size="0.8128" layer="25" font="vector" rot="R180"/>
 <attribute name="VALUE" x="12.3608" y="18.0312" size="0.4064" layer="27" font="vector" rot="R180"/>
