File: hardware/riffle-beta-0.1.0/riffle-beta-0.1.8.5.sch (EAGLE design)
At the start: 51 parts, among them IC1 ATMEGA328P, IC3 CH340G, IC4 MCP1700-33, IC5 24AA128SN, IC6 MCP1700-33, J1 AYZ0202, U1 MCP73831T-2ACI/OT, X2 12MHz, X3 16 MHz

Commit message: update
Parts:
- C2: value 0.1uF -> 10uF
Changed lines of the file:
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@@
 <part name="R10" library="microbuilder" deviceset="RESISTOR" device="_0603_NOOUT" value="1.4K"/>
 <part name="C1" library="SparkFun" deviceset="CAP" device="0603-CAP" value="10uF"/>
-<part name="C2" library="SparkFun" deviceset="CAP" device="0603-CAP" value="0.1uF"/>
+<part name="C2" library="SparkFun" deviceset="CAP" device="0603-CAP" value="10uF"/>
 <part name="C3" library="SparkFun" deviceset="CAP" device="0603-CAP" value="0.1uF"/>
 <part name="C4" library="SparkFun" deviceset="CAP" device="0603-CAP" value="10uF"/>
